Commit message: Exercises

File: dev_ws/src/minibot/urdf/minibot_base.xacro (robot description, xacro)
@@ -1,4 +1,5 @@
 <?xml version="1.0"?>
-<robot name="minibot_base" xmlns:xacro="http://www.ros.org/wiki/xacro">
+<!-- <robot name="minibot_base" xmlns:xacro="http://www.ros.org/wiki/xacro"> -->
+<robot xmlns:xacro="http://www.ros.org/wiki/xacro" >
         <!-- colors -->
         <material name="white">
@@ -68,5 +69,5 @@
                 <child link="right_wheel_link"/>
                 <origin xyz="${wheel_offset_x} ${-((chassis_width/2) + (wheel_thickness/2))} 0" rpy="${pi/2} 0 0"/>
-                <axis xyz="0 0 1"/>
+                <axis xyz="0 0 -1"/>
         </joint>
         <!-- right_wheel_link -->
